Commit message: Fix hardware interface to work with real robot

File: src/thor_description/urdf/thor.xacro (robot description, xacro)
@@ -1,9 +1,9 @@
-<?xml version="1.0" ?>
+<?xml version="1.0"?>
 <robot name="thor" xmlns:xacro="http://www.ros.org/wiki/xacro">
     <xacro:include filename="$(find thor_description)/urdf/thor.gazebo" />
     <link name="dummy_link" />
     <joint name="dummy_joint" type="fixed">
-        <parent link="dummy_link"/>
-        <child link="link_base"/>
+        <parent link="dummy_link" />
+        <child link="link_base" />
     </joint>
     <link name="link_base">
@@ -25,11 +25,11 @@
     </link>
     <joint name="joint_base_art1_yaw" type="revolute">
-      <origin xyz="0 0 0.104" rpy="0 0 0"/>
-      <axis xyz="0 0 1"/>
-      <parent link="link_base"/>
-      <child link="link_art1"/>
-      <limit lower="-3.1415" upper="3.1415" effort="4" velocity="1" />
+        <origin xyz="0 0 0.104" rpy="0 0 0" />
+        <axis xyz="0 0 1" />
+        <parent link="link_base" />
+        <child link="link_art1" />
+        <limit lower="-3.1415" upper="3.1415" effort="4" velocity="1" />
     </joint>
-     <link name="link_art1">
+    <link name="link_art1">
         <collision>
             <origin xyz="0 0 0" rpy="0 0 0" />
@@ -41,5 +41,6 @@
             <origin xyz="0 0 0" rpy="0 0 0" />
             <geometry>
-                <mesh filename="package://thor_description/meshes/art1.stl" scale="0.001 0.001 0.001" />
+                <mesh filename="package://thor_description/meshes/art1.stl"
+                    scale="0.001 0.001 0.001" />
             </geometry>
             <material name="black">
@@ -49,9 +50,9 @@
     </link>
     <joint name="joint_art1_art2_pitch" type="revolute">
-        <origin xyz="0 -0.0318752 0.0974304" rpy="1.5707963267948966 -1.5707963267948966 0"/>
-	<axis xyz="0 0 1"/>
-	<parent link="link_art1"/>
-        <child link="link_art2"/>
-	<limit lower="-1.5707963267948966" upper="1.5707963267948966" effort="4" velocity="1" />
+        <origin xyz="0 -0.0318752 0.0974304" rpy="1.5707963267948966 -1.5707963267948966 0" />
+        <axis xyz="0 0 1" />
+        <parent link="link_art1" />
+        <child link="link_art2" />
+        <limit lower="-1.5707963267948966" upper="1.5707963267948966" effort="4" velocity="1" />
     </joint>
     <link name="link_art2">
@@ -71,12 +72,12 @@
     </link>
     <joint name="joint_art2_art3_pitch" type="revolute">
-        <origin xyz="0.160 0 0" rpy="0 0 0"/>
-	<axis xyz="0 0 1"/>
-	<parent link="link_art2"/>
-        <child link="link_art3"/>
-	<limit lower="-1.5707963267948966" upper="1.5707963267948966" effort="4" velocity="1" />
+        <origin xyz="0.160 0 0" rpy="0 0 0" />
+        <axis xyz="0 0 1" />
+        <parent link="link_art2" />
+        <child link="link_art3" />
+        <limit lower="-1.5707963267948966" upper="1.5707963267948966" effort="4" velocity="1" />
     </joint>
     <link name="link_art3">
-    	<collision>
+        <collision>
             <origin xyz="0 0 0" rpy="0 0 0" />
             <geometry>
@@ -93,15 +94,16 @@
     </link>
     <joint name="joint_art3_art4_roll" type="revolute">
-        <origin xyz="0.0885 0 -0.035" rpy="0 1.5707963267948966 0"/>
-	<axis xyz="0 0 1"/>
-	<parent link="link_art3"/>
-        <child link="link_art4"/>
-	<limit lower="-3.1415" upper="3.1415" effort="4" velocity="1" />
+        <origin xyz="0.0885 0 -0.035" rpy="0 1.5707963267948966 0" />
+        <axis xyz="0 0 1" />
+        <parent link="link_art3" />
+        <child link="link_art4" />
+        <limit lower="-3.1415" upper="3.1415" effort="4" velocity="1" />
     </joint>
     <link name="link_art4">
-    	<collision>
+        <collision>
             <origin xyz="0 0 0" rpy="0 0 0" />
             <geometry>
-                <mesh filename="package://thor_description/meshes/art4.stl" scale="0.001 0.001 0.001" />
+                <mesh filename="package://thor_description/meshes/art4.stl"
+                    scale="0.001 0.001 0.001" />
             </geometry>
         </collision>
@@ -109,5 +111,6 @@
             <origin xyz="0 0 0" rpy="0 0 0" />
             <geometry>
-                <mesh filename="package://thor_description/meshes/art4.stl" scale="0.001 0.001 0.001" />
+                <mesh filename="package://thor_description/meshes/art4.stl"
+                    scale="0.001 0.001 0.001" />
             </geometry>
             <material name="brown" />
@@ -115,15 +118,16 @@
     </link>
     <joint name="joint_art4_art5_pitch" type="revolute">
-        <origin xyz="0 0 0.1" rpy="0 -1.5707963267948966 0"/>
-	<axis xyz="0 0 1"/>
-	<parent link="link_art4"/>
-        <child link="link_art5"/>
-	<limit lower="-1.5" upper="1.5" effort="4" velocity="1" />
+        <origin xyz="0 0 0.1" rpy="0 -1.5707963267948966 0" />
+        <axis xyz="0 0 1" />
+        <parent link="link_art4" />
+        <child link="link_art5" />
+        <limit lower="-1.5" upper="1.5" effort="4" velocity="1" />
     </joint>
     <link name="link_art5">
-    	<collision>
+        <collision>
             <origin xyz="0 0 0" rpy="0 0 0" />
             <geometry>
-                <mesh filename="package://thor_description/meshes/art5.stl" scale="0.001 0.001 0.001" />
+                <mesh filename="package://thor_description/meshes/art5.stl"
+                    scale="0.001 0.001 0.001" />
             </geometry>
         </collision>
@@ -131,5 +135,6 @@
             <origin xyz="0 0 0" rpy="0 0 0" />
             <geometry>
-                <mesh filename="package://thor_description/meshes/art5.stl" scale="0.001 0.001 0.001" />
+                <mesh filename="package://thor_description/meshes/art5.stl"
+                    scale="0.001 0.001 0.001" />
             </geometry>
             <material name="black" />
@@ -137,15 +142,16 @@
     </link>
     <joint name="joint_art5_art6_roll" type="revolute">
-        <origin xyz="0 0 0" rpy="0 1.5707963267948966 0"/>
-	<axis xyz="0 0 1"/>
-	<parent link="link_art5"/>
-        <child link="link_art6"/>
-	<limit lower="-3.1415" upper="3.1415" effort="4" velocity="1" />
+        <origin xyz="0 0 0" rpy="0 1.5707963267948966 0" />
+        <axis xyz="0 0 1" />
+        <parent link="link_art5" />
+        <child link="link_art6" />
+        <limit lower="-3.1415" upper="3.1415" effort="4" velocity="1" />
     </joint>
     <link name="link_art6">
-    	<collision>
+        <collision>
             <origin xyz="0 0 0" rpy="0 0 0" />
             <geometry>
-                <mesh filename="package://thor_description/meshes/art6.stl" scale="0.001 0.001 0.001" />
+                <mesh filename="package://thor_description/meshes/art6.stl"
+                    scale="0.001 0.001 0.001" />
             </geometry>
         </collision>
@@ -153,5 +159,6 @@
             <origin xyz="0 0 0" rpy="0 0 0" />
             <geometry>
-                <mesh filename="package://thor_description/meshes/art6.stl" scale="0.001 0.001 0.001" />
+                <mesh filename="package://thor_description/meshes/art6.stl"
+                    scale="0.001 0.001 0.001" />
             </geometry>
             <material name="black" />

File: src/thor_moveit/config/gazebo_thor.urdf (robot description, URDF)
Before this commit: robot thor, 8 links, 7 joints
Links:
- link link_base: mass 0.1 -> 10

Commit message: Add gripper to urdf

File: src/thor_description/urdf/thor.xacro (robot description, xacro)
@@ -19,6 +19,6 @@
                 <mesh filename="package://thor_description/meshes/base.stl" scale="0.001 0.001 0.001" />
             </geometry>
-            <material name="brown">
-                <color rgba="0.369 0.216 0 1" />
+            <material name="white">
+                <color rgba="1 1 1 1" />
             </material>
         </visual>
@@ -45,5 +45,5 @@
             </geometry>
             <material name="black">
-                <color rgba="0.1 0.1 0.1 1" />
+                <color rgba="0.4 0.4 0.4 1" />
             </material>
         </visual>
@@ -68,5 +68,5 @@
                 <mesh filename="package://thor_description/meshes/art2.stl" scale="0.001 0.001 0.001" />
             </geometry>
-            <material name="brown" />
+            <material name="white" />
         </visual>
     </link>
@@ -114,5 +114,5 @@
                     scale="0.001 0.001 0.001" />
             </geometry>
-            <material name="brown" />
+            <material name="white" />
         </visual>
     </link>
@@ -165,3 +165,76 @@
         </visual>
     </link>
+    <joint name="joint_arm_hand" type="fixed">
+        <origin xyz="0 0.015 0.07" rpy="1.5707963267948966 0 0"  />
+        <parent link="link_art6" />
+        <child link="link_hand" />
+    </joint>
+    <link name="link_hand">
+        <collision>
+            <origin xyz="0 0 0" rpy="0 0 0" />
+            <geometry>
+                <mesh filename="package://thor_description/meshes/hand.stl"
+                    scale="0.001 0.001 0.001" />
+            </geometry>
+        </collision>
+        <visual>
+            <origin xyz="0 0 0" rpy="0 0 0" />
+            <geometry>
+                <mesh filename="package://thor_description/meshes/hand.stl"
+                    scale="0.001 0.001 0.001" />
+            </geometry>
+            <material name="black" />
+        </visual>
+    </link>
+    <joint name="joint_hand_finger_left" type="prismatic">
+        <parent link="link_hand" />
+        <child link="link_finger_left" />
+        <origin rpy="0 0 0" xyz="0.05 0.02 0" />
+        <axis xyz="-1 1.5 0" />
+        <limit effort="100" lower="0.0" upper="0.03" velocity="0.2" />
+        <dynamics damping="0.3" />
+    </joint>
+    <joint name="joint_hand_finger_right" type="prismatic">
+        <parent link="link_hand" />
+        <child link="link_finger_right" />
+        <origin rpy="0 0 0" xyz="-0.05 0.02 0" />
+        <axis xyz="1 1.5 0" />
+        <limit effort="100" lower="0.0" upper="0.03" velocity="0.2" />
+        <mimic joint="joint_hand_finger_left" />
+        <dynamics damping="0.3" />
+    </joint>
+    <link name="link_finger_left">
+        <collision>
+            <origin xyz="0 0 0." rpy="0 0 0" />
+            <geometry>
+                <mesh filename="package://thor_description/meshes/finger.stl"
+                    scale="-0.001 0.001 0.001" />
+            </geometry>
+        </collision>
+        <visual>
+            <origin xyz="0 0 0" rpy="0 0 0" />
+            <geometry>
+                <mesh filename="package://thor_description/meshes/finger.stl"
+                    scale="-0.001 0.001 0.001" />
+            </geometry>
+            <material name="white" />
+        </visual>
+    </link>
+    <link name="link_finger_right">
+        <collision>
+            <origin xyz="0 0 0" rpy="0 0 0" />
+            <geometry>
+                <mesh filename="package://thor_description/meshes/finger.stl"
+                    scale="0.001 0.001 0.001" />
+            </geometry>
+        </collision>
+        <visual>
+            <origin xyz="0 0 0" rpy="0 0 0" />
+            <geometry>
+                <mesh filename="package://thor_description/meshes/finger.stl"
+                    scale="0.001 0.001 0.001" />
+            </geometry>
+            <material name="white" />
+        </visual>
+    </link>
 </robot>

File: src/thor_moveit/config/gazebo_thor.urdf (robot description, URDF)
Before this commit: robot thor, 8 links, 7 joints
Links:
- added link link_finger_left, mass 0.1; collision mesh filename=package://thor_description/meshes/finger.stl scale=-0.001 0.001 0.001; visual mesh filename=package://thor_description/meshes/finger.stl scale=-0.001 0.001 0.001
- added link link_finger_right, mass 0.1; collision mesh filename=package://thor_description/meshes/finger.stl scale=0.001 0.001 0.001; visual mesh filename=package://thor_description/meshes/finger.stl scale=0.001 0.001 0.001
- added link link_hand, mass 0.1; collision mesh filename=package://thor_description/meshes/hand.stl scale=0.001 0.001 0.001; visual mesh filename=package://thor_description/meshes/hand.stl scale=0.001 0.001 0.001
- link link_base: mass 10 -> 0.1
Joints:
- added joint joint_arm_hand: type fixed, parent link_art6, child link_hand, origin xyz=0 0.015 0.07 rpy=1.5707963267948966 0 0
- added joint joint_hand_finger_left: type prismatic, parent link_hand, child link_finger_left, origin xyz=0.05 0.02 0 rpy=0 0 0, axis -1 1.5 0, limit lower=0.0 upper=0.03 effort=100 velocity=0.2
- added joint joint_hand_finger_right: type prismatic, parent link_hand, child link_finger_right, origin xyz=-0.05 0.02 0 rpy=0 0 0, axis 1 1.5 0, limit lower=0.0 upper=0.03 effort=100 velocity=0.2, mimic joint=joint_hand_finger_left

Commit message: Add gripper controller

File: src/thor_description/urdf/thor.xacro (robot description, xacro)
@@ -192,5 +192,5 @@
         <origin rpy="0 0 0" xyz="0.05 0.02 0" />
         <axis xyz="-1 1.5 0" />
-        <limit effort="100" lower="0.0" upper="0.03" velocity="0.2" />
+        <limit effort="100" lower="0.0" upper="0.03" velocity="10" />
         <dynamics damping="0.3" />
     </joint>
@@ -200,5 +200,5 @@
         <origin rpy="0 0 0" xyz="-0.05 0.02 0" />
         <axis xyz="1 1.5 0" />
-        <limit effort="100" lower="0.0" upper="0.03" velocity="0.2" />
+        <limit effort="100" lower="0.0" upper="0.03" velocity="10" />
         <mimic joint="joint_hand_finger_left" />
         <dynamics damping="0.3" />

File: src/thor_moveit/config/gazebo_thor.urdf (robot description, URDF)
Before this commit: robot thor, 11 links, 10 joints
Joints:
- joint joint_hand_finger_left: limit lower=0.0 upper=0.03 effort=100 velocity=0.2 -> lower=0.0 upper=0.03 effort=100 velocity=10
- joint joint_hand_finger_right: limit lower=0.0 upper=0.03 effort=100 velocity=0.2 -> lower=0.0 upper=0.03 effort=100 velocity=10

Commit message: Add inertia to urdf

File: src/thor_description/urdf/thor.xacro (robot description, xacro)
@@ -23,4 +23,8 @@
             </material>
         </visual>
+        <inertial>
+            <mass value="20" />
+            <inertia ixx="0.03" iyy="0.03" izz="0.03" ixy="0.0" ixz="0.0" iyz="0.0" />
+        </inertial>
     </link>
     <joint name="joint_base_art1_yaw" type="revolute">
@@ -48,4 +52,8 @@
             </material>
         </visual>
+        <inertial>
+            <mass value="1.6" />
+            <inertia ixx="0.03" iyy="0.03" izz="0.03" ixy="0.0" ixz="0.0" iyz="0.0" />
+        </inertial>
     </link>
     <joint name="joint_art1_art2_pitch" type="revolute">
@@ -70,4 +78,8 @@
             <material name="white" />
         </visual>
+        <inertial>
+            <mass value="0.8" />
+            <inertia ixx="0.03" iyy="0.03" izz="0.03" ixy="0.0" ixz="0.0" iyz="0.0" />
+        </inertial>
     </link>
     <joint name="joint_art2_art3_pitch" type="revolute">
@@ -92,4 +104,8 @@
             <material name="black" />
         </visual>
+        <inertial>
+            <mass value="1.1" />
+            <inertia ixx="0.03" iyy="0.03" izz="0.03" ixy="0.0" ixz="0.0" iyz="0.0" />
+        </inertial>
     </link>
     <joint name="joint_art3_art4_roll" type="revolute">
@@ -116,4 +132,8 @@
             <material name="white" />
         </visual>
+        <inertial>
+            <mass value="0.5" />
+            <inertia ixx="0.03" iyy="0.03" izz="0.03" ixy="0.0" ixz="0.0" iyz="0.0" />
+        </inertial>
     </link>
     <joint name="joint_art4_art5_pitch" type="revolute">
@@ -140,4 +160,8 @@
             <material name="black" />
         </visual>
+        <inertial>
+            <mass value="0.5" />
+            <inertia ixx="0.03" iyy="0.03" izz="0.03" ixy="0.0" ixz="0.0" iyz="0.0" />
+        </inertial>
     </link>
     <joint name="joint_art5_art6_roll" type="revolute">
@@ -164,4 +188,8 @@
             <material name="black" />
         </visual>
+        <inertial>
+            <mass value="0.5" />
+            <inertia ixx="0.03" iyy="0.03" izz="0.03" ixy="0.0" ixz="0.0" iyz="0.0" />
+        </inertial>
     </link>
     <joint name="joint_arm_hand" type="fixed">

File: src/thor_moveit/config/gazebo_thor.urdf (robot description, URDF)
Before this commit: robot thor, 11 links, 10 joints
Links:
- link link_art1: mass 0.1 -> 1.6
- link link_art2: mass 0.1 -> 0.8
- link link_art3: mass 0.1 -> 1.1
- link link_art4: mass 0.1 -> 0.5
- link link_art5: mass 0.1 -> 0.5
- link link_art6: mass 0.1 -> 0.5
- link link_base: mass 0.1 -> 20

Commit message: Fix pid and effort for gazebo

File: src/thor_description/urdf/thor.xacro (robot description, xacro)
@@ -33,5 +33,5 @@
         <parent link="link_base" />
         <child link="link_art1" />
-        <limit lower="-3.1415" upper="3.1415" effort="4" velocity="1" />
+        <limit lower="-3.1415" upper="3.1415" effort="8" velocity="1" />
     </joint>
     <link name="link_art1">
@@ -62,5 +62,5 @@
         <parent link="link_art1" />
         <child link="link_art2" />
-        <limit lower="-1.5707963267948966" upper="1.5707963267948966" effort="4" velocity="1" />
+        <limit lower="-1.5707963267948966" upper="1.5707963267948966" effort="20" velocity="1" />
     </joint>
     <link name="link_art2">
@@ -88,5 +88,5 @@
         <parent link="link_art2" />
         <child link="link_art3" />
-        <limit lower="-1.5707963267948966" upper="1.5707963267948966" effort="4" velocity="1" />
+        <limit lower="-1.5707963267948966" upper="1.5707963267948966" effort="8" velocity="1" />
     </joint>
     <link name="link_art3">
@@ -142,5 +142,5 @@
         <parent link="link_art4" />
         <child link="link_art5" />
-        <limit lower="-1.5" upper="1.5" effort="4" velocity="1" />
+        <limit lower="-1.5" upper="1.5" effort="6" velocity="1" />
     </joint>
     <link name="link_art5">

File: src/thor_moveit/config/gazebo_thor.urdf (robot description, URDF)
Before this commit: robot thor, 11 links, 10 joints
Joints:
- joint joint_art1_art2_pitch: limit lower=-1.5707963267948966 upper=1.5707963267948966 effort=4 velocity=1 -> lower=-1.5707963267948966 upper=1.5707963267948966 effort=20 velocity=1
- joint joint_art2_art3_pitch: limit lower=-1.5707963267948966 upper=1.5707963267948966 effort=4 velocity=1 -> lower=-1.5707963267948966 upper=1.5707963267948966 effort=8 velocity=1
- joint joint_art4_art5_pitch: limit lower=-1.5 upper=1.5 effort=4 velocity=1 -> lower=-1.5 upper=1.5 effort=6 velocity=1
- joint joint_base_art1_yaw: limit lower=-3.1415 upper=3.1415 effort=4 velocity=1 -> lower=-3.1415 upper=3.1415 effort=8 velocity=1

Commit message: Fix bug gripper move by normalizing vectors

File: src/thor_description/urdf/thor.xacro (robot description, xacro)
@@ -219,6 +219,6 @@
         <child link="link_finger_left" />
         <origin rpy="0 0 0" xyz="0.05 0.02 0" />
-        <axis xyz="-1 1.5 0" />
-        <limit effort="100" lower="0.0" upper="0.03" velocity="10" />
+        <axis xyz="-0.5547 0.8321 0"/>
+        <limit effort="100" lower="0.0" upper="0.06" velocity="10" />
         <dynamics damping="0.3" />
     </joint>
@@ -227,6 +227,6 @@
         <child link="link_finger_right" />
         <origin rpy="0 0 0" xyz="-0.05 0.02 0" />
-        <axis xyz="1 1.5 0" />
-        <limit effort="100" lower="0.0" upper="0.03" velocity="10" />
+        <axis xyz="0.5547 0.8321 0"/>
+        <limit effort="100" lower="0.0" upper="0.06" velocity="10" />
         <mimic joint="joint_hand_finger_left" />
         <dynamics damping="0.3" />

File: src/thor_moveit/config/gazebo_thor.urdf (robot description, URDF)
Before this commit: robot thor, 11 links, 10 joints
Joints:
- joint joint_hand_finger_left: axis -1 1.5 0 -> -0.5547 0.8321 0; limit lower=0.0 upper=0.03 effort=100 velocity=10 -> lower=0.0 upper=0.06 effort=100 velocity=10
- joint joint_hand_finger_right: axis 1 1.5 0 -> 0.5547 0.8321 0; limit lower=0.0 upper=0.03 effort=100 velocity=10 -> lower=0.0 upper=0.06 effort=100 velocity=10
