Commit message: Update thor description with complete parts

File: src/thor_description/urdf/gazebo.xacro (robot description, xacro)
@@ -26,5 +26,14 @@
     </gazebo>
     <gazebo reference="link_art6">
-        <material>Gazebo/Black</material>
+      <material>Gazebo/Black</material>
+    </gazebo>
+    <gazebo reference="link_hand">
+      <material>Gazebo/Black</material>
+    </gazebo>
+    <gazebo reference="link_finger_left">
+      <material>Gazebo/White</material>
+    </gazebo>
+    <gazebo reference="link_finger_right">
+      <material>Gazebo/White</material>
     </gazebo>
     <xacro:macro name="gazebo_mimic_joint_plugin" params="name_prefix parent_joint mimic_joint has_pid:=false multiplier:=1.0 offset:=0 sensitiveness:=0.0 max_effort:=1.0 robot_namespace:=''">

File: src/thor_description/urdf/thor.xacro (robot description, xacro)
@@ -25,5 +25,5 @@
         <inertial>
             <mass value="20" />
-            <inertia ixx="0.03" iyy="0.03" izz="0.03" ixy="0.0" ixz="0.0" iyz="0.0" />
+            <inertia ixx="4778335232" iyy="9956602880" izz="12350248960" ixy="61676072" ixz="-346234336" iyz="-3673513" />
         </inertial>
     </link>
@@ -54,5 +54,5 @@
         <inertial>
             <mass value="1.6" />
-            <inertia ixx="0.03" iyy="0.03" izz="0.03" ixy="0.0" ixz="0.0" iyz="0.0" />
+            <inertia ixx="2091996160" iyy="2178797312" izz="1449157760" ixy="-6433.202148" ixz="-9487.117188" iyz="96796960" />
         </inertial>
     </link>
@@ -80,5 +80,5 @@
         <inertial>
             <mass value="0.8" />
-            <inertia ixx="0.03" iyy="0.03" izz="0.03" ixy="0.0" ixz="0.0" iyz="0.0" />
+            <inertia ixx="2494758144" iyy="5296528896" izz="4277223680" ixy="169831.156250" ixz="-192684608" iyz="-4347370" />l
         </inertial>
     </link>
@@ -106,5 +106,5 @@
         <inertial>
             <mass value="1.1" />
-            <inertia ixx="0.03" iyy="0.03" izz="0.03" ixy="0.0" ixz="0.0" iyz="0.0" />
+            <inertia ixx="509821408" iyy="861984512" izz="946194816" ixy="-4423478.5" ixz="1108099" iyz="-62569.3125" />
         </inertial>
     </link>
@@ -134,5 +134,5 @@
         <inertial>
             <mass value="0.5" />
-            <inertia ixx="0.03" iyy="0.03" izz="0.03" ixy="0.0" ixz="0.0" iyz="0.0" />
+            <inertia ixx="766526720" iyy="898525120" izz="718228096" ixy="513188.25" ixz="-15419.867188" iyz="546204.625" />
         </inertial>
     </link>
@@ -162,5 +162,5 @@
         <inertial>
             <mass value="0.5" />
-            <inertia ixx="0.03" iyy="0.03" izz="0.03" ixy="0.0" ixz="0.0" iyz="0.0" />
+            <inertia ixx="22853730" iyy="16640192" izz="36724072" ixy="-103.737335" ixz="-10548.656250" iyz="-0.059193" />
         </inertial>
     </link>
@@ -190,5 +190,5 @@
         <inertial>
             <mass value="0.5" />
-            <inertia ixx="0.03" iyy="0.03" izz="0.03" ixy="0.0" ixz="0.0" iyz="0.0" />
+            <inertia ixx="33753776" iyy="33753756" izz="24939260" ixy="-2.472111" ixz="-21.388384" iyz="0.078231" />
         </inertial>
     </link>
@@ -214,4 +214,8 @@
             <material name="black" />
         </visual>
+        <inertial>
+            <mass value="0.11" />
+            <inertia ixx="17803724" iyy="21783168" izz="28014524" ixy="-414543.5" ixz="225471.4375" iyz="-1840743.875" />
+        </inertial>
     </link>
     <joint name="joint_hand_finger_left" type="prismatic">
@@ -221,5 +225,5 @@
         <axis xyz="-0.5547 0.8321 0"/>
         <limit effort="100" lower="0.0" upper="0.06" velocity="10" />
-        <dynamics damping="0.3" />
+        <dynamics damping="0.3" friction="0.5" />
     </joint>
     <joint name="joint_hand_finger_right" type="prismatic">
@@ -230,12 +234,12 @@
         <limit effort="100" lower="0.0" upper="0.06" velocity="10" />
         <mimic joint="joint_hand_finger_left" />
-        <dynamics damping="0.3" />
+        <dynamics damping="0.3" friction="0.5" />
     </joint>
     <xacro:gazebo_mimic_joint_plugin name_prefix="joint_hand_finger_right"
         parent_joint="joint_hand_finger_left" mimic_joint="joint_hand_finger_right"
-        has_pid="true" />
+        has_pid="false" />
     <link name="link_finger_left">
         <collision>
-            <origin xyz="0 0 0." rpy="0 0 0" />
+            <origin xyz="0 0 0" rpy="0 0 0" />
             <geometry>
                 <mesh filename="package://thor_description/meshes/finger.stl"
@@ -251,4 +255,8 @@
             <material name="white" />
         </visual>
+        <inertial>
+            <mass value="0.01" />
+            <inertia ixx="3358780.25" iyy="627437.875" izz="3410634.5" ixy="-145110.265625" ixz="93.539124" iyz="1280.361816" />
+        </inertial>
     </link>
     <link name="link_finger_right">
@@ -268,4 +276,8 @@
             <material name="white" />
         </visual>
+        <inertial>
+            <mass value="0.01" />
+            <inertia ixx="3358780.25" iyy="627437.875" izz="3410634.5" ixy="-145110.265625" ixz="93.539124" iyz="1280.361816" />
+        </inertial>
     </link>
 </robot>

File: src/thor_moveit/config/gazebo_thor.urdf (robot description, URDF)
Before this commit: robot thor, 11 links, 10 joints
Links:
- link link_finger_left: mass 0.1 -> 0.01
- link link_finger_right: mass 0.1 -> 0.01
- link link_hand: mass 0.1 -> 0.11

Commit message: Add env in urdf

File: src/thor_description/urdf/gazebo.xacro (robot description, xacro)
@@ -38,20 +38,20 @@
     </gazebo>
     <xacro:macro name="gazebo_mimic_joint_plugin" params="name_prefix parent_joint mimic_joint has_pid:=false multiplier:=1.0 offset:=0 sensitiveness:=0.0 max_effort:=1.0 robot_namespace:=''">
-    <gazebo>
-      <plugin name="${name_prefix}_mimic_joint_plugin" filename="libroboticsgroup_upatras_gazebo_mimic_joint_plugin.so">
-        <joint>${parent_joint}</joint>
-        <mimicJoint>${mimic_joint}</mimicJoint>
-        <xacro:if value="${has_pid}"> <!-- if set to true, PID parameters from "/gazebo_ros_control/pid_gains/${mimic_joint}" are loaded -->
-          <hasPID />
-        </xacro:if>
-        <multiplier>${multiplier}</multiplier>
-        <offset>${offset}</offset>
-        <sensitiveness>${sensitiveness}</sensitiveness>
-        <maxEffort>${max_effort}</maxEffort>
-        <xacro:unless value="${robot_namespace == ''}">
-          <robotNamespace>${robot_namespace}</robotNamespace>
-        </xacro:unless>
-      </plugin>
-    </gazebo>
-  </xacro:macro>
+        <gazebo>
+            <plugin name="${name_prefix}_mimic_joint_plugin" filename="libroboticsgroup_upatras_gazebo_mimic_joint_plugin.so">
+                <joint>${parent_joint}</joint>
+                <mimicJoint>${mimic_joint}</mimicJoint>
+                <xacro:if value="${has_pid}"> <!-- if set to true, PID parameters from "/gazebo_ros_control/pid_gains/${mimic_joint}" are loaded -->
+                    <hasPID />
+                </xacro:if>
+                <multiplier>${multiplier}</multiplier>
+                <offset>${offset}</offset>
+                <sensitiveness>${sensitiveness}</sensitiveness>
+                <maxEffort>${max_effort}</maxEffort>
+                <xacro:unless value="${robot_namespace == ''}">
+                    <robotNamespace>${robot_namespace}</robotNamespace>
+                </xacro:unless>
+            </plugin>
+        </gazebo>
+    </xacro:macro>
 </robot>

File: src/thor_description/urdf/thor.xacro (robot description, xacro)
@@ -2,6 +2,8 @@
 <robot name="thor" xmlns:xacro="http://www.ros.org/wiki/xacro">
     <xacro:include filename="$(find thor_description)/urdf/gazebo.xacro" />
+    <xacro:include filename="$(find thor_description)/urdf/env.xacro" />
     <link name="dummy_link" />
     <joint name="dummy_joint" type="fixed">
+        <origin xyz="0.1 0 0" rpy="0 0 0"/>   <!-- move thor a bit forward on the counter -->
         <parent link="dummy_link" />
         <child link="link_base" />

File: src/thor_moveit/config/gazebo_thor.urdf (robot description, URDF)
Before this commit: robot thor, 11 links, 10 joints
Links:
- added link counter, mass 0.1; collision box size=0.59 0.38 0.1; visual box size=0.59 0.38 0.1
- added link roof, mass 0.1; collision box size=0.6 1.02 0.42; visual box size=0.6 1.02 0.42
- added link stove, mass 0.1; collision box size=0.59 0.64 0.1; visual box size=0.59 0.64 0.1
- added link wall_back, mass 0.1; collision box size=0.1 1.02 1; visual box size=0.1 1.02 1
- added link wall_left, mass 0.1; collision box size=0.59 0.1 1; visual box size=0.59 0.1 1
Joints:
- added joint joint_counter: type fixed, parent dummy_link, child counter, origin xyz=0 0 -0.05 rpy=0 0 0
- added joint joint_roof: type fixed, parent dummy_link, child roof, origin xyz=-0.3 0.32 0.79 rpy=0 0 0
- added joint joint_stove: type fixed, parent dummy_link, child stove, origin xyz=0 0.51 -0.05 rpy=0 0 0
- added joint joint_wall_back: type fixed, parent dummy_link, child wall_back, origin xyz=-0.345 0.32 0.5 rpy=0 0 0
- added joint joint_wall_left: type fixed, parent dummy_link, child wall_left, origin xyz=0 -0.24 0.5 rpy=0 0 0
- joint dummy_joint: origin (none) -> xyz=0.1 0 0 rpy=0 0 0
